File: touch-circuit-v2/touch-circuit-v2.kicad_pcb (KiCad board)
At the start: 2 copper layers, 18.7 x 20.5 mm, 11 parts, among them Q1 NMOS, Q2 PMOS

Commit message: update back silk
Parts:
- added REF**: TY_Mark_3mm_Silkscreen, #footprints:TY_Mark_3mm_Silkscreen, B.Cu at (148.8, 91.4)
Routing:
- net GND: track 0.00 -> 33.8 mm
- net Net-(BT1-Pad1): track 43.4 -> 42.1 mm
- net /Gate: track 34.4 -> 35.7 mm
Changed lines of the file:
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@@
     (thickness 1.6)
     (drawings 6)
-    (tracks 64)
+    (tracks 75)
     (zones 0)
-    (modules 11)
+    (modules 12)
     (nets 8)
   )
   (page A4)
   (layers
-    (0 F.Cu signal)
+    (0 F.Cu signal hide)
     (31 B.Cu signal)
     (32 B.Adhes user hide)
@@
     (35 F.Paste user hide)
     (36 B.SilkS user)
-    (37 F.SilkS user)
+    (37 F.SilkS user hide)
     (38 B.Mask user)
-    (39 F.Mask user)
+    (39 F.Mask user hide)
     (40 Dwgs.User user hide)
     (41 Cmts.User user hide)
@@
     (44 Edge.Cuts user)
     (45 Margin user hide)
-    (46 B.CrtYd user)
-    (47 F.CrtYd user)
-    (48 B.Fab user)
-    (49 F.Fab user)
+    (46 B.CrtYd user hide)
+    (47 F.CrtYd user hide)
+    (48 B.Fab user hide)
+    (49 F.Fab user hide)
   )
   (setup
@@
       (outputformat 1)
       (mirror false)
-      (drillshape 1)
+      (drillshape 0)
       (scaleselection 1)
-      (outputdirectory ""))
+      (outputdirectory "gerber"))
   )
   (net 0 "")
@@
     (add_net "Net-(D1-Pad2)")
     (add_net "Net-(Q1-Pad3)")
+  )
+  (module "#footprints:TY_Mark_3mm_Silkscreen" (layer B.Cu)
+    (at 148.844 91.44 180)
+    (fp_text reference REF** (at 0 5 180) (layer B.SilkS) hide
+      (effects (font (size 1 1) (thickness 0.15)) (justify mirror))
+    )
+    (fp_text value TY_Mark_3mm_Silkscreen (at 0 -4.5 180) (layer B.Fab) hide
+      (effects (font (size 1 1) (thickness 0.15)) (justify mirror))
+    )
+    (fp_poly (pts (xy -1.075 0.85) (xy -1.6 1.175) (xy -1.35 1.175) (xy -1.175 0.925)) (layer B.SilkS) (width 0.08))
+    (fp_poly (pts (xy 0.425 1.05) (xy 0.5 1.175) (xy 0.275 1.175) (xy 0.275 1.125)) (layer B.SilkS) (width 0.08))
+    (fp_poly (pts (xy -0.625 -1.1) (xy -0.425 -0.8) (xy -0.45 -1) (xy -0.5 -1)) (layer B.SilkS) (width 0.08))
+    (fp_poly (pts (xy 0.35 0.15) (xy 0.55 0.45) (xy 0.55 0.25) (xy 0.5 0.25)) (layer B.SilkS) (width 0.08))
+    (fp_line (start -1.4 1.125) (end 0.35 1.125) (layer B.SilkS) (width 0.18))
+    (fp_line (start -0.5 1.7) (end -0.5 0.15) (layer B.SilkS) (width 0.18))
+    (fp_line (start 0.5 0.25) (end 0.5 -1) (layer B.SilkS) (width 0.18))
+    (fp_arc (start 0 -1) (end -0.5 -1) (angle 180) (layer B.SilkS) (width 0.18))
+    (fp_arc (start 0 0.15) (end -0.5 0.15) (angle 180) (layer B.SilkS) (width 0.18))
+    (fp_poly (pts (xy -0.65 1.6) (xy -0.45 1.9) (xy -0.45 1.7) (xy -0.5 1.7)) (layer B.SilkS) (width 0.08))
   )
   (module "#footprints:WireMount" (layer F.Cu)
@@
     )
   )
-  (gr_line (start 137.668 98.044) (end 133.604 93.98) (layer Edge.Cuts) (width 0.15))
-  (gr_line (start 137.668 101.6) (end 137.668 98.044) (layer Edge.Cuts) (width 0.15))
-  (gr_line (start 146.812 98.044) (end 150.876 93.98) (layer Edge.Cuts) (width 0.15))
-  (gr_line (start 146.812 101.6) (end 146.812 98.044) (layer Edge.Cuts) (width 0.15))
-  (gr_line (start 137.668 101.6) (end 146.812 101.6) (layer Edge.Cuts) (width 0.15))
-  (gr_arc (start 142.24 90.424) (end 150.876 93.98) (angle -224.7602701) (layer Edge.Cuts) (width 0.15))
+  (gr_line (start 137.668 98.044) (end 133.604 93.98) (layer Edge.Cuts) (width 0.0254))
+  (gr_line (start 137.668 101.6) (end 137.668 98.044) (layer Edge.Cuts) (width 0.0254))
+  (gr_line (start 146.812 98.044) (end 150.876 93.98) (layer Edge.Cuts) (width 0.0254))
+  (gr_line (start 146.812 101.6) (end 146.812 98.044) (layer Edge.Cuts) (width 0.0254))
+  (gr_line (start 137.668 101.6) (end 146.812 101.6) (layer Edge.Cuts) (width 0.0254))
+  (gr_arc (start 142.24 90.424) (end 150.876 93.98) (angle -224.7602701) (layer Edge.Cuts) (width 0.0254))
   (segment (start 144.502 89.94) (end 145.354 89.94) (width 0.25) (layer F.Cu) (net 1))
   (segment (start 143.256 91.186) (end 144.502 89.94) (width 0.25) (layer F.Cu) (net 1))
@@
   (segment (start 142.24 98.61) (end 142.56501 98.93501) (width 0.25) (layer F.Cu) (net 1))
   (segment (start 142.24 98.035) (end 142.24 98.61) (width 0.25) (layer F.Cu) (net 1))
-  (segment (start 145.136999 99.211001) (end 142.24 99.211001) (width 0.25) (layer B.Cu) (net 1))
-  (segment (start 145.542 98.806) (end 145.136999 99.211001) (width 0.25) (layer B.Cu) (net 1))
-  (segment (start 145.542 96.52) (end 145.542 98.806) (width 0.25) (layer B.Cu) (net 1))
-  (segment (start 140.94 84.011001) (end 142.24 84.011001) (width 0.25) (layer B.Cu) (net 1))
-  (segment (start 136.814999 88.136002) (end 140.94 84.011001) (width 0.25) (layer B.Cu) (net 1))
-  (segment (start 136.814999 96.586) (end 136.814999 88.136002) (width 0.25) (layer B.Cu) (net 1))
-  (segment (start 139.44 99.211001) (end 136.814999 96.586) (width 0.25) (layer B.Cu) (net 1))
-  (segment (start 142.24 99.211001) (end 139.44 99.211001) (width 0.25) (layer B.Cu) (net 1))
   (segment (start 143.374 92.447) (end 143.256 92.447) (width 0.25) (layer F.Cu) (net 1))
   (segment (start 144.78 93.853) (end 143.374 92.447) (width 0.25) (layer F.Cu) (net 1))
   (segment (start 144.78 95.758) (end 144.78 93.853) (width 0.25) (layer F.Cu) (net 1))
   (segment (start 145.542 96.52) (end 144.78 95.758) (width 0.25) (layer F.Cu) (net 1))
-  (via (at 147.828 86.36) (size 0.8) (drill 0.4) (layers F.Cu B.Cu) (net 2))
-  (via (at 136.652 86.36) (size 0.8) (drill 0.4) (layers F.Cu B.Cu) (net 2))
+  (segment (start 143.612999 99.211001) (end 142.24 99.211001) (width 0.25) (layer B.Cu) (net 1))
+  (segment (start 145.542 97.282) (end 143.612999 99.211001) (width 0.25) (layer B.Cu) (net 1))
+  (segment (start 145.542 96.52) (end 145.542 97.282) (width 0.25) (layer B.Cu) (net 1))
+  (segment (start 140.94 84.011001) (end 142.24 84.011001) (width 0.25) (layer B.Cu) (net 1))
+  (segment (start 136.814999 95.793999) (end 136.814999 88.136002) (width 0.25) (layer B.Cu) (net 1))
+  (segment (start 138.266001 97.245001) (end 136.814999 95.793999) (width 0.25) (layer B.Cu) (net 1))
+  (segment (start 136.814999 88.136002) (end 140.94 84.011001) (width 0.25) (layer B.Cu) (net 1))
+  (segment (start 139.028001 97.245001) (end 138.266001 97.245001) (width 0.25) (layer B.Cu) (net 1))
+  (segment (start 140.994001 99.211001) (end 139.028001 97.245001) (width 0.25) (layer B.Cu) (net 1))
+  (segment (start 142.24 99.211001) (end 140.994001 99.211001) (width 0.25) (layer B.Cu) (net 1))
   (via (at 138.938 96.52) (size 0.8) (drill 0.4) (layers F.Cu B.Cu) (net 2))
+  (via (at 134.62 88.9) (size 0.8) (drill 0.4) (layers F.Cu B.Cu) (net 2))
+  (via (at 149.86 88.9) (size 0.8) (drill 0.4) (layers F.Cu B.Cu) (net 2))
+  (segment (start 149.86 94.2975) (end 149.86 90.932) (width 0.25) (layer B.Cu) (net 2))
+  (segment (start 149.86 90.932) (end 149.86 88.9) (width 0.25) (layer B.Cu) (net 2))
+  (segment (start 146.05 98.1075) (end 149.86 94.2975) (width 0.25) (layer B.Cu) (net 2))
+  (segment (start 146.05 100.076) (end 146.05 98.1075) (width 0.25) (layer B.Cu) (net 2))
+  (segment (start 145.288 100.838) (end 146.05 100.076) (width 0.25) (layer B.Cu) (net 2))
+  (segment (start 138.43 100.076) (end 139.192 100.838) (width 0.25) (layer B.Cu) (net 2))
+  (segment (start 138.43 98.07865) (end 138.43 100.076) (width 0.25) (layer B.Cu) (net 2))
+  (segment (start 134.62 94.26865) (end 138.43 98.07865) (width 0.25) (layer B.Cu) (net 2))
+  (segment (start 139.192 100.838) (end 145.288 100.838) (width 0.25) (layer B.Cu) (net 2))
+  (segment (start 134.62 88.9) (end 134.62 94.26865) (width 0.25) (layer B.Cu) (net 2))
   (segment (start 141.224 86.369) (end 141.215 86.36) (width 0.25) (layer F.Cu) (net 3))
   (segment (start 141.224 92.447) (end 141.224 86.369) (width 0.25) (layer F.Cu) (net 3))
@@
   (segment (start 139 100.085) (end 138.06801 99.15301) (width 0.25) (layer F.Cu) (net 7))
   (segment (start 139.7 100.085) (end 139 100.085) (width 0.25) (layer F.Cu) (net 7))
-  (segment (start 136.056001 85.685999) (end 135.109949 86.632051) (width 0.25) (layer F.Cu) (net 7))
-  (segment (start 136.906 84.836) (end 136.056001 85.685999) (width 0.25) (layer F.Cu) (net 7))
-  (segment (start 148.405948 85.667948) (end 149.352 86.614) (width 0.25) (layer F.Cu) (net 7))
-  (segment (start 147.555949 84.817949) (end 148.405948 85.667948) (width 0.25) (layer F.Cu) (net 7))
-  (segment (start 147.537898 84.836) (end 147.555949 84.817949) (width 0.25) (layer F.Cu) (net 7))
-  (segment (start 136.906 84.836) (end 147.537898 84.836) (width 0.25) (layer F.Cu) (net 7))
   (segment (start 139.126 88.58) (end 139.126 89.94) (width 0.25) (layer F.Cu) (net 7))
   (segment (start 138.176 87.63) (end 139.126 88.58) (width 0.25) (layer F.Cu) (net 7))
   (segment (start 136.107898 87.63) (end 138.176 87.63) (width 0.25) (layer F.Cu) (net 7))
   (segment (start 135.109949 86.632051) (end 136.107898 87.63) (width 0.25) (layer F.Cu) (net 7))
+  (segment (start 135.109949 86.632051) (end 136.906 84.836) (width 0.25) (layer B.Cu) (net 7))
+  (segment (start 147.555949 84.817949) (end 149.352 86.614) (width 0.25) (layer B.Cu) (net 7))
+  (segment (start 146.05 83.312) (end 147.555949 84.817949) (width 0.25) (layer F.Cu) (net 7))
+  (segment (start 138.43 83.312) (end 146.05 83.312) (width 0.25) (layer F.Cu) (net 7))
+  (segment (start 136.906 84.836) (end 138.43 83.312) (width 0.25) (layer F.Cu) (net 7))
   (zone (net 2) (net_name GND) (layer F.Cu) (hatch edge 0.508)
     (connect_pads (clearance 0.508))
